File: DesignFiles/POV2.3.brd (EAGLE design)
At the start: 99.2 x 49.6 mm, 27 parts, among them CN1 1X4-CLEANBIG, CN2 1X4-CLEANBIG, CN3 1X4-CLEANBIG, CN4 1X4-CLEANBIG, J1 PINHD-1X10, J2 PINHD-1X10

Commit message: Some logo tweaks to the board
Parts:
- added U$7, U$8: (no value), 43oh_logo:CIRCUIT_LOG_STOP_ONLY
Changed lines of the file:
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@@
 </element>
 <element name="U$3" library="TIBadgeCustom" package="BADGE_BACK_REVERSE" value="" x="0.127" y="0.254"/>
+<element name="U$7" library="43oh_logo" package="CIRCUIT_LOG_STOP_ONLY" value="" x="5.9436" y="16.9672" rot="MR270"/>
+<element name="U$8" library="43oh_logo" package="CIRCUIT_LOG_STOP_ONLY" value="" x="67.5132" y="6.8072" rot="MR180"/>
 </elements>
 <signals>
